File: RM27_Accu_TS_Schematic.kicad_sch (KiCad schematic)
At the start: 22 parts, among them SW1 HV+, SW2 HV-

Commit message: Updated new maintenance plugs for mr trimper
Parts:
- SW? (x5): value MaintenancePlug -> 2X MaintenancePlug
- SW?: value MaintentancePlug -> 2X MaintentancePlug
